Commit message: Docs: RViz successfully running with arm_group configuration

File: robot_arm_simulation/urdf/robot_arm_urdf.xacro (robot description, xacro)
@@ -220,11 +220,32 @@
       <plugin>gz_ros2_control/GazeboSimSystem</plugin>
     </hardware>
-    <joint name="joint_1"><command_interface name="position"/><state_interface name="position"/></joint>
-    <joint name="joint_2"><command_interface name="position"/><state_interface name="position"/></joint>
-    <joint name="joint_3"><command_interface name="position"/><state_interface name="position"/></joint>
-    <joint name="joint_4"><command_interface name="position"/><state_interface name="position"/></joint>
-    <joint name="joint_5"><command_interface name="position"/><state_interface name="position"/></joint>
-    <joint name="joint_6"><command_interface name="position"/><state_interface name="position"/></joint>
-    <joint name="joint_7"><command_interface name="position"/><state_interface name="position"/></joint>
+    <joint name="joint_1">
+      <command_interface name="position"/>
+      <state_interface name="position"/>
+      <state_interface name="velocity"/> </joint>
+    <joint name="joint_2">
+      <command_interface name="position"/>
+      <state_interface name="position"/>
+      <state_interface name="velocity"/> </joint>
+    <joint name="joint_3">
+      <command_interface name="position"/>
+      <state_interface name="position"/>
+      <state_interface name="velocity"/> </joint>
+    <joint name="joint_4">
+      <command_interface name="position"/>
+      <state_interface name="position"/>
+      <state_interface name="velocity"/> </joint>
+    <joint name="joint_5">
+      <command_interface name="position"/>
+      <state_interface name="position"/>
+      <state_interface name="velocity"/> </joint>
+    <joint name="joint_6">
+      <command_interface name="position"/>
+      <state_interface name="position"/>
+      <state_interface name="velocity"/> </joint>
+    <joint name="joint_7">
+      <command_interface name="position"/>
+      <state_interface name="position"/>
+      <state_interface name="velocity"/> </joint>
   </ros2_control>
   <gazebo>
